File: SOURCES/FreeDSP_SMD.kicad_pcb (KiCad board)
At the start: 2 copper layers, 100 x 100 mm, 187 parts, among them IC1 AD8608ARZ, IC2 ADAU1701, IC3 24AA256, IC4 SN74LVC1G08DBVR, IC5 AD8608ARZ, IC6 AD8608ARZ, IC7 74HC4040D, P10 CONN_02X10, P11 MM-16G, P12 MM-12G, P2 BARREL_JACK, P3 CONN_02X02, P4 USBi, P5 CONN_02X13, P6 CONN_01X06, P7 CONN_01X06, P8 CONN_01X06, P9 CONN_02X10, Q1 ZXTP25040DFHTA, Q2 2N7000, Q3 2N7000, U1 78033, U3 7805

Commit message: WB on GND
Connections:
- IC2 pad 20: (no net) -> GND
Routing:
- net GND: track 16.8 -> 33.5 mm, vias 5 -> 6
- net (no net): track 7.80 -> 0.00 mm
- net /WP: track 47.2 -> 50.0 mm
- net /OUT2: track 3.90 -> 5.70 mm
- net +5V: track 330.4 -> 329.4 mm
Changed lines of the file:
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@@
 (kicad_pcb (version 4) (host pcbnew 4.0.2-stable)
   (general
-    (links 415)
-    (no_connects 4)
-    (area 93.224999 49.949999 205.300001 150.050001)
+    (links 416)
+    (no_connects 0)
+    (area 99.949999 49.949999 200.050001 150.050001)
     (thickness 1.6)
     (drawings 13)
-    (tracks 1334)
+    (tracks 1344)
     (zones 0)
     (modules 187)
@@
     (tags 0805)
     (attr smd)
-    (fp_text reference R5 (at 0 -2.1 180) (layer F.SilkS)
+    (fp_text reference R5 (at 0 1.7 180) (layer F.SilkS)
       (effects (font (size 1 1) (thickness 0.15)))
     )
@@
     (pad 19 smd rect (at 0.25 4.35 180) (size 1.3 0.25) (layers F.Cu F.Paste F.Mask)
       (net 42 MP11))
-    (pad 20 smd rect (at 0.75 4.35 180) (size 1.3 0.25) (layers F.Cu F.Paste F.Mask))
+    (pad 20 smd rect (at 0.75 4.35 180) (size 1.3 0.25) (layers F.Cu F.Paste F.Mask)
+      (net 1 GND))
     (pad 21 smd rect (at 1.25 4.35 180) (size 1.3 0.25) (layers F.Cu F.Paste F.Mask)
       (net 21 /WP))
@@
     (effects (font (size 0.8 0.8) (thickness 0.2)) (justify left))
   )
-  (segment (start 176.664426 95.5) (end 177.539437 94.624989) (width 0.25) (layer F.Cu) (net 0))
-  (segment (start 176.664426 95.5) (end 174.414426 97.75) (width 0.25) (layer F.Cu) (net 0))
-  (segment (start 177.239437 94.924989) (end 176.664426 95.5) (width 0.25) (layer F.Cu) (net 0))
-  (segment (start 174.414426 97.75) (end 171.85 97.75) (width 0.25) (layer F.Cu) (net 0))
+  (via (at 180.135 125.565) (size 1.8) (drill 0.9) (layers F.Cu B.Cu) (net 1))
+  (segment (start 180.135 123.4) (end 180.135 125.565) (width 0.25) (layer F.Cu) (net 1))
+  (segment (start 182.9 101.5) (end 183.8 101.5) (width 0.25) (layer F.Cu) (net 1))
+  (segment (start 183.8 101.5) (end 184.8 102.5) (width 0.25) (layer F.Cu) (net 1))
+  (segment (start 176.664426 95.5) (end 177.989447 94.174979) (width 0.25) (layer F.Cu) (net 1))
+  (segment (start 177.989447 94.174979) (end 181.865021 94.174979) (width 0.25) (layer F.Cu) (net 1))
+  (segment (start 181.865021 94.174979) (end 182.424001 93.615999) (width 0.25) (layer F.Cu) (net 1))
+  (segment (start 182.424001 93.615999) (end 183.44 92.6) (width 0.25) (layer F.Cu) (net 1))
+  (segment (start 176.664426 95.5) (end 174.414426 97.75) (width 0.25) (layer F.Cu) (net 1))
+  (segment (start 177.239437 94.924989) (end 176.664426 95.5) (width 0.25) (layer F.Cu) (net 1))
+  (segment (start 174.414426 97.75) (end 171.85 97.75) (width 0.25) (layer F.Cu) (net 1))
   (segment (start 182.9 98.3) (end 185.143138 98.3) (width 0.25) (layer F.Cu) (net 1))
   (segment (start 185.143138 98.3) (end 185.208987 98.234151) (width 0.25) (layer F.Cu) (net 1))
@@
   (segment (start 144.4 84.6) (end 150.3 84.6) (width 0.25) (layer F.Cu) (net 1))
   (via (at 150.3 84.6) (size 1.8) (drill 0.9) (layers F.Cu B.Cu) (net 1))
-  (segment (start 182.9 101.5) (end 183.8 101.5) (width 0.25) (layer F.Cu) (net 1))
-  (segment (start 183.8 101.5) (end 184.8 102.5) (width 0.25) (layer F.Cu) (net 1))
   (via (at 184.8 102.5) (size 1.8) (drill 0.9) (layers F.Cu B.Cu) (net 1))
   (segment (start 170.25 94.15) (end 171.35 94.15) (width 0.25) (layer F.Cu) (net 1))
@@
   (segment (start 177.6 104.9) (end 177.6 103.2972) (width 0.25) (layer F.Cu) (net 20))
   (segment (start 177.6 103.2972) (end 177.55 103.2472) (width 0.25) (layer F.Cu) (net 20))
+  (segment (start 182.299997 108.512999) (end 182.1 108.313002) (width 0.25) (layer B.Cu) (net 21))
+  (segment (start 182.1 108.313002) (end 179.9 106.113002) (width 0.25) (layer B.Cu) (net 21))
+  (segment (start 182.4 108.613002) (end 182.1 108.313002) (width 0.25) (layer B.Cu) (net 21))
+  (segment (start 173.3 97.25) (end 174.278016 97.25) (width 0.25) (layer F.Cu) (net 21))
+  (segment (start 172.8 97.25) (end 173.3 97.25) (width 0.25) (layer F.Cu) (net 21))
+  (segment (start 173.3 97.25) (end 171.85 97.25) (width 0.25) (layer F.Cu) (net 21))
+  (segment (start 182.9 96.3) (end 184.7 96.3) (width 0.25) (layer F.Cu) (net 21))
+  (segment (start 178.865 118) (end 178.865 116.975) (width 0.25) (layer F.Cu) (net 21))
+  (segment (start 178.865 116.975) (end 179.420011 116.419989) (width 0.25) (layer F.Cu) (net 21))
+  (segment (start 179.420011 116.419989) (end 180.980011 116.419989) (width 0.25) (layer F.Cu) (net 21))
+  (segment (start 180.980011 116.419989) (end 182.4 115) (width 0.25) (layer F.Cu) (net 21))
+  (segment (start 182.4 115) (end 182.4 113.7) (width 0.25) (layer F.Cu) (net 21))
+  (segment (start 182.4 113.7) (end 182.4 112.4) (width 0.25) (layer F.Cu) (net 21))
   (segment (start 184.7 96.3) (end 181 92.6) (width 0.25) (layer B.Cu) (net 21))
   (segment (start 181 92.6) (end 180.9 92.6) (width 0.25) (layer B.Cu) (net 21))
   (segment (start 182.4 108.613002) (end 182.4 112.4) (width 0.25) (layer B.Cu) (net 21))
-  (segment (start 178.895 117.495) (end 179.970011 116.419989) (width 0.25) (layer F.Cu) (net 21))
-  (segment (start 179.970011 116.419989) (end 181.052213 116.419989) (width 0.25) (layer F.Cu) (net 21))
   (segment (start 182.3 112.5) (end 182.4 112.4) (width 0.25) (layer F.Cu) (net 21))
-  (segment (start 181.052213 116.419989) (end 182.299997 115.172205) (width 0.25) (layer F.Cu) (net 21))
-  (segment (start 182.299997 115.172205) (end 182.299997 113.700003) (width 0.25) (layer F.Cu) (net 21))
-  (segment (start 182.299997 113.700003) (end 182.3 113.7) (width 0.25) (layer F.Cu) (net 21))
-  (segment (start 182.3 113.7) (end 182.3 112.5) (width 0.25) (layer F.Cu) (net 21))
   (segment (start 178.865 117.525) (end 178.865 118) (width 0.25) (layer F.Cu) (net 21))
   (segment (start 182.299997 112.299997) (end 182.3 112.3) (width 0.25) (layer B.Cu) (net 21))
   (via (at 182.4 112.4) (size 1.8) (drill 0.9) (layers F.Cu B.Cu) (net 21))
-  (segment (start 182.299997 108.512999) (end 179.9 106.113002) (width 0.25) (layer B.Cu) (net 21))
   (segment (start 179.9 106.113002) (end 179.9 105.086998) (width 0.25) (layer B.Cu) (net 21))
   (segment (start 184.7 96.3) (end 183.474999 97.525001) (width 0.25) (layer B.Cu) (net 21))
@@
   (segment (start 176.928016 94.6) (end 178.528016 93) (width 0.25) (layer F.Cu) (net 21))
   (segment (start 178.528016 93) (end 180.9 93) (width 0.25) (layer F.Cu) (net 21))
-  (segment (start 182.9 96.3) (end 184.7 96.3) (width 0.25) (layer F.Cu) (net 21))
   (via (at 184.7 96.3) (size 1.8) (drill 0.9) (layers F.Cu B.Cu) (net 21))
   (segment (start 174.278016 97.25) (end 176.928016 94.6) (width 0.25) (layer F.Cu) (net 21))
@@
   (segment (start 172.8 97.25) (end 171.85 97.25) (width 0.25) (layer F.Cu) (net 21))
   (segment (start 173.145519 97.25) (end 172.8 97.25) (width 0.25) (layer F.Cu) (net 21))
-  (segment (start 172.8 97.25) (end 174.278016 97.25) (width 0.25) (layer F.Cu) (net 21))
   (segment (start 168.15 87.95) (end 168.6 88.4) (width 0.25) (layer F.Cu) (net 22))
   (segment (start 168.6 88.4) (end 168.6 88.9) (width 0.25) (layer F.Cu) (net 22))
@@
   (segment (start 176.912 67.739732) (end 176.906 67.745732) (width 0.25) (layer F.Cu) (net 28))
   (segment (start 174.106 67.739732) (end 174.112 67.745732) (width 0.25) (layer F.Cu) (net 28))
+  (segment (start 137.8 52) (end 169.2 52) (width 0.6) (layer B.Cu) (net 29))
+  (segment (start 169.2 59.4) (end 169.198 59.402) (width 0.6) (layer F.Cu) (net 29))
+  (segment (start 169.198 59.402) (end 167.086 59.402) (width 0.6) (layer F.Cu) (net 29))
   (segment (start 189.863601 120.2) (end 189.863601 137.638817) (width 0.6) (layer F.Cu) (net 29))
   (segment (start 189.863601 119.323601) (end 189.863601 120.2) (width 0.6) (layer F.Cu) (net 29))
@@
   (segment (start 137.8 66.8) (end 141.1 70.1) (width 0.6) (layer F.Cu) (net 29))
   (segment (start 174 59.4) (end 169.2 59.4) (width 0.6) (layer F.Cu) (net 29))
-  (segment (start 169.2 59.4) (end 167.088 59.4) (width 0.6) (layer F.Cu) (net 29))
   (segment (start 169.2 52) (end 169.2 59.4) (width 0.6) (layer F.Cu) (net 29))
-  (segment (start 139.072792 52) (end 170.2 52) (width 0.6) (layer B.Cu) (net 29))
   (via (at 169.2 52) (size 1.8) (drill 0.9) (layers F.Cu B.Cu) (net 29))
-  (segment (start 137.8 52) (end 139.072792 52) (width 0.6) (layer B.Cu) (net 29))
   (segment (start 137.8 66.8) (end 137.8 52) (width 0.6) (layer F.Cu) (net 29))
   (via (at 137.8 52) (size 1.8) (drill 0.9) (layers F.Cu B.Cu) (net 29))
@@
   (segment (start 126.5 62.6) (end 126.5 64.7) (width 0.25) (layer F.Cu) (net 52))
   (segment (start 124.7 62.6) (end 126.5 62.6) (width 0.25) (layer F.Cu) (net 52))
+  (segment (start 124.7 74.3) (end 126.5 74.3) (width 0.25) (layer F.Cu) (net 53))
   (segment (start 126.5 74.3) (end 126.5 76.4) (width 0.25) (layer F.Cu) (net 53))
   (segment (start 124.7 76.4) (end 126.5 76.4) (width 0.25) (layer F.Cu) (net 53))
