File: SOURCES/FreeDSP_SMD.sch (KiCad schematic (older format))
At the start: 163 parts, among them IC1 AD8608, IC2 ADAU1701, IC3 24AA256, IC4 TC7SZ08, IC5 AD8608, IC6 AD8608, P1 CONN_02X11, P10 CONN_02X10, P2 CONN_2, P3 CONN_02X02, P4 USBi, P5 CONN_02X13, P6 CONN_01X06, P7 CONN_01X06, P8 CONN_01X06, P9 CONN_02X10, Q1 PNP, Q2 2N7000, Q3 2N7000, U1 78033, U2 4040, U3 7805, X1 12M288Hz

Commit message: Cleaned BOM (footprints).
Parts:
- C1, C17, C23: footprint Capacitors_SMD:C_0805 -> rklib:C0805-X7R
- C11, C14, C21, C22, C24, C25, C9: value 10u -> 10u0; footprint Capacitors_SMD:C_0805 -> rklib:C0805-X7R
- C18: value 10n -> 10n0; footprint Capacitors_SMD:C_0805 -> rklib:C0805-X7R
- C19, C20, C36, C37: value 3n3 -> 3n30
- C30: value 3n3 -> 3n30; footprint Capacitors_SMD:C_0805 -> rklib:C0805-X7R
- C31: value 56n -> 56n0; footprint Capacitors_SMD:C_0805 -> rklib:C0805-X7R
- C32, C33: value 22p -> 22p0; footprint Capacitors_SMD:C_0805 -> rklib:C0805-X7R
- Q1: value PNP -> ZXTP25040DFHTA
- R1, R15, R16, R18, R19, R2, R3, R4: value 4k75 -> 4K75
- R10, R11, R26, R27: value 47k -> 47K0
- R12, R13, R14, R9: value 18k -> 18K0
- R17: value 1k -> 1K00; footprint Resistors_SMD:R_0805 -> rklib:C0805-RES
- R20, R21: footprint Resistors_SMD:R_0805 -> rklib:C0805-RES
- R22, R23, R7, R8: value 680 -> 680R
- R24, R25: value 10k -> 10K0; footprint Resistors_SMD:R_0805 -> rklib:C0805-RES
- R28, R36, R37, R45, R46, R47, R52, R53, R58, R59, R64, R65, R71, R75: value 10k -> 10K0
- R29, R34, R38, R43: value 100k -> 100K
- R31, R33, R40, R42: value 20k -> 20K0
- R49, R55, R61, R67: value 22k -> 22K0

Commit message: - Added 10K PullUp and GND-Jumper on WP-line - Fixed footprint of Q1
Parts:
- added JP4: JUMPER, Pin_Headers:Pin_Header_Straight_1x02, symbol JUMPER
- added R5: 10K0, rklib:C0805-RES, symbol R-RESCUE-FreeDSP_SMD
Connections:
- wire segments 220 -> 224
Other:
- moved on the sheet: C11, C14, C17, C38, C39, C4, C40, C8, C9, IC1E, IC3, JP1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

Commit message: - Bugfix ADC-Stage: Applied VCC/2 - Changed VCC of OpAmps to +5V - Changed gains, Pro: +6dBu (ARD-Norm) and Con: -10dBv for full scale
Parts:
- removed IC5: AD8608, Housings_SOIC:SOIC-14_3.9x8.7mm_Pitch1.27mm, symbol OPAMP4
- added C10, C7: 47u0./16V, Capacitors_ThroughHole:C_Radial_D5_L11_P2, symbol CP
- added IC5: AD8608ARZ, Housings_SOIC:SOIC-14_3.9x8.7mm_Pitch1.27mm, symbol AD8608ARZ
- added R77, R78: 47K0, rklib:C0805-RES, symbol R-RESCUE-FreeDSP_SMD
- C43, C44, C50, C51: value 47u0 ./ 35V -> 47u0./35V
- R13, R14: value 18K0 -> 7K15
- R31, R33, R40, R42: value 20K0 -> 17K4
- R35, R44: value 100R -> 3K57
Connections:
- net labels added: Vcom
- wire segments 224 -> 238
Other:
- moved on the sheet: B1, B2, B3, B4, C1, C18, C21, C22, C23, C24, C25, C30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

Commit message: Bugfix DAC-Stage: Applied VCC/2 - Supplied OpAmps with +5V - Reworked gain settings: Pro +6dBu, Consumer -10dBV
Parts:
- removed C55, C57, C59, C62: 47u0 ./ 35V, Capacitors_ThroughHole:C_Radial_D8_L11.5_P3.5, symbol C-RESCUE-FreeDSP_SMD
- removed IC1, IC6: AD8608, Housings_SOIC:SOIC-14_3.9x8.7mm_Pitch1.27mm, symbol OPAMP4
- added C12, C13, C15, C16, C34, C35, C55, C57, C59, C62, C63, C64: 47u0./16V, Capacitors_ThroughHole:C_Radial_D5_L11_P2, symbol CP
- added IC1, IC6: AD8608ARZ, Housings_SOIC:SOIC-14_3.9x8.7mm_Pitch1.27mm, symbol AD8608ARZ
- added JP5, JP6, JP7, JP8: JUMPER3, Pin_Headers:Pin_Header_Straight_1x03, symbol JUMPER3
- added R79, R80, R81, R82: 17K4, rklib:C0805-RES, symbol R-RESCUE-FreeDSP_SMD
- R10, R11: value 47K0 -> 49K9
- R46, R52, R58, R64: value 10K0 -> 3K57
- R7, R8: value 680R -> 604R
Connections:
- wire segments 238 -> 260
Other:
- note added: "TODO 100n hinzufügen"
- moved on the sheet: C19, C2, C20, C26, C27, C28, C29, C3, C36, C37, C39, C5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

Commit message: Changed DC supply connector to barrel jack
Parts:
- removed C4, C8: 220u, Capacitors_ThroughHole:C_Radial_D10_L13_P5, symbol CAPAPOL
- removed P2: CONN_2, Connect:bornier2, symbol CONN_2
- added C4, C8: 220u./35V, Capacitors_ThroughHole:C_Radial_D10_L13_P5, symbol CP
- added C65: 100n, rklib:C0805-X7R, symbol C-RESCUE-FreeDSP_SMD
- added P2: BARREL_JACK, Connect:BARREL_JACK, symbol BARREL_JACK
Connections:
- net +5V: now also C4.1
- net 3V3: now also C8.1
- net GND: now also C4.2, C65.1, C8.2, P2.2, P2.3
- net at C14.1, U3.VI: now also P2.1
- net at IC5.5 (+), R77.2, R78.1: now also C65.2
Other:
- note added: "<= 1%"
- note added: "POWER"
- note removed: "<= 1% Toleranze"
- note removed: "TODO 100n hinzufügen"
- moved on the sheet: B1, B2, B3, B4, C1, C11, C18, C21, C22, C23, C24, C25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

Commit message: Changed expansion header to new standard i2s expansion header
Parts:
- removed IC4: TC7SZ08, TO_SOT_Packages_SMD:SOT-23-5, symbol TC7SZ08
- removed P1: CONN_02X11, Pin_Headers:Pin_Header_Straight_2x11, symbol CONN_02X11
- removed U2: 4040, Housings_SOIC:SOIC-16_3.9x9.9mm_Pitch1.27mm, symbol 4040
- added IC4: SN74LVC1G08DBVR, TO_SOT_Packages_SMD:SOT-23-5, symbol SN74LVC1G08DBVR
- added IC7: 74HC4040D, Housings_SOIC:SOIC-16_3.9x9.9mm_Pitch1.27mm, symbol 74HC4040D
- added P11: MM-16G, rklib:MM-16G, symbol CONN_01X16
- added P12: MM-12G, rklib:MM-12G, symbol CONN_01X12
- renumbered X1 to OSC1
Connections:
- net WB is gone; now on net GND: IC2.20 (ADDR1/CDATA/WB)
- net +5V: now also P12.1 (P1); no longer JP1.2
- net 3V3: now also IC4.5 (Vcc), IC7.16 (VDD)
- net GND: now also IC4.3 (GND), IC7.11 (Reset), IC7.8 (VSS), P11.10 (P10), P11.12 (P12), P11.14 (P14), P11.16 (P16), P11.2 (P2), P11.4 (P4), P11.6 (P6), P11.8 (P8), P12.12 (P12), P12.2 (P2)
- net IN1: now also IC2.2 (ADC0), R13.2; no longer C7.2, R13.1
- net IN2: now also IC2.4 (ADC1), R14.2; no longer C10.2, R14.1
- net MCLK: now also P11.15 (P15)
- net MP0: now also P11.3 (P3)
- net MP1: now also P12.6 (P6)
- net MP10: now also P11.9 (P9)
- net MP11: now also P11.7 (P7)
- net MP2: now also P12.11 (P11)
- net MP3: now also P12.10 (P10)
- net MP4: now also P12.4 (P4)
- net MP5: now also P12.5 (P5)
- net MP6: now also P11.5 (P5)
- net MP7: now also P12.7 (P7)
- net MP8: now also P12.9 (P9)
- net MP9: now also P12.8 (P8)
- net SCL: now also P11.13 (P13)
- net SDA: now also P11.11 (P11)
- net _RESET: now also P12.3 (P3)
- net at IC2.31 (OSCO), R21.1: now also IC4.1 (B), IC4.2 (A)
- net at JP1.1: now also P11.1 (P1)
- net at P5.25 (P25): now also IC7.1 (Q11)
- net at P5.1 (P1): now also IC4.4 (Y), IC7.10 (CLK)
- net at P5.19 (P19): now also IC7.12 (Q8)
- net at P5.17 (P17): now also IC7.13 (Q7)
- net at P5.21 (P21): now also IC7.14 (Q9)
- net at P5.23 (P23): now also IC7.15 (Q10)
- net at P5.13 (P13): now also IC7.2 (Q5)
- net at P5.11 (P11): now also IC7.3 (Q4)
- net at P5.15 (P15): now also IC7.4 (Q6)
- net at P5.9 (P9): now also IC7.5 (Q3)
- net at P5.7 (P7): now also IC7.6 (Q2)
- net at P5.5 (P5): now also IC7.7 (Q1)
- net at P5.3 (P3): now also IC7.9 (Q0)
- net VCC: now reaches C14.1, P2.1, U3.VI
- net VCC: now also JP1.2
- new net: C7.2, R13.1
- new net: C10.2, R14.1
Other:
- moved on the sheet: C1, C11, C14, C17, C18, C21, C22, C23, C24, C25, C30, C31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

Commit message: WB on GND
Other:
- moved on the sheet: JP1, P11, P12
Changed lines of the file:
@@
 L JUMPER JP1
 U 1 1 566A6CA5
-P 16050 2400
-F 0 "JP1" H 16050 2550 50  0000 C CNN
-F 1 "JUMPER" H 16050 2320 50  0000 C CNN
-F 2 "Pin_Headers:Pin_Header_Straight_1x02" H 16050 2400 60  0001 C CNN
-F 3 "" H 16050 2400 60  0000 C CNN
-	1    16050 2400
+P 1050 4050
+F 0 "JP1" H 1050 4200 50  0000 C CNN
+F 1 "JUMPER" H 1050 3970 50  0000 C CNN
+F 2 "Pin_Headers:Pin_Header_Straight_1x02" H 1050 4050 60  0001 C CNN
+F 3 "" H 1050 4050 60  0000 C CNN
+	1    1050 4050
 	1    0    0    -1
 $EndComp
@@
 L CONN_01X16 P11
 U 1 1 5745D956
-P 15550 3150
-F 0 "P11" H 15550 4000 50  0000 C CNN
-F 1 "MM-16G" V 15650 3150 50  0000 C CNN
-F 2 "rklib:MM-16G" H 15550 3150 50  0001 C CNN
-F 3 "" H 15550 3150 50  0000 C CNN
-	1    15550 3150
+P 550 4800
+F 0 "P11" H 550 5650 50  0000 C CNN
+F 1 "MM-16G" H 450 3900 50  0000 C CNN
+F 2 "rklib:MM-16G" H 550 4800 50  0001 C CNN
+F 3 "" H 550 4800 50  0000 C CNN
+	1    550  4800
 	-1   0    0    -1
 $EndComp
@@
 Connection ~ 4800 3600
 Wire Wire Line
-	15750 2500 15850 2500
+	750  4150 850  4150
 Wire Wire Line
-	15850 2500 15850 4000
+	850  4150 850  5650
 $Comp
 L GND-RESCUE-FreeDSP_SMD #PWR0111
 U 1 1 57477E35
-P 15850 4000
-F 0 "#PWR0111" H 15850 4000 30  0001 C CNN
-F 1 "GND" H 15850 3930 30  0001 C CNN
-F 2 "" H 15850 4000 60  0000 C CNN
-F 3 "" H 15850 4000 60  0000 C CNN
-	1    15850 4000
+P 850 5650
+F 0 "#PWR0111" H 850 5650 30  0001 C CNN
+F 1 "GND" H 850 5580 30  0001 C CNN
+F 2 "" H 850 5650 60  0000 C CNN
+F 3 "" H 850 5650 60  0000 C CNN
+	1    850  5650
 	1    0    0    -1
 $EndComp
-Text GLabel 17350 750  2    47   Input ~ 0
+Text GLabel 1100 1350 2    47   Input ~ 0
 _RESET
-Text GLabel 17350 950  2    47   Input ~ 0
+Text GLabel 1100 1550 2    47   Input ~ 0
 MP5
-Text GLabel 15900 2600 2    47   Input ~ 0
+Text GLabel 900  4250 2    47   Input ~ 0
 MP0
-Text GLabel 15900 2800 2    47   Input ~ 0
+Text GLabel 900  4450 2    47   Input ~ 0
 MP6
-Text GLabel 15900 3000 2    47   Input ~ 0
+Text GLabel 900  4650 2    47   Input ~ 0
 MP11
-Text GLabel 15900 3600 2    47   Input ~ 0
+Text GLabel 900  5250 2    47   Input ~ 0
 SCL
-Text GLabel 17350 1350 2    47   Input ~ 0
+Text GLabel 1100 1950 2    47   Input ~ 0
 MP8
-Text GLabel 15900 3800 2    47   Input ~ 0
+Text GLabel 900  5450 2    47   Input ~ 0
 MCLK
-Text GLabel 17350 1550 2    47   Input ~ 0
+Text GLabel 1100 2150 2    47   Input ~ 0
 MP2
-Text GLabel 17350 1450 2    47   Input ~ 0
+Text GLabel 1100 2050 2    47   Input ~ 0
 MP3
-Text GLabel 17350 1250 2    47   Input ~ 0
+Text GLabel 1100 1850 2    47   Input ~ 0
 MP9
-Text GLabel 15900 3400 2    47   Input ~ 0
+Text GLabel 900  5050 2    47   Input ~ 0
 SDA
-Text GLabel 15900 3200 2    47   Input ~ 0
+Text GLabel 900  4850 2    47   Input ~ 0
 MP10
-Text GLabel 17350 1150 2    47   Input ~ 0
+Text GLabel 1100 1750 2    47   Input ~ 0
 MP7
-Text GLabel 17350 1050 2    47   Input ~ 0
+Text GLabel 1100 1650 2    47   Input ~ 0
 MP1
-Text GLabel 17350 850  2    47   Input ~ 0
+Text GLabel 1100 1450 2    47   Input ~ 0
 MP4
 Wire Wire Line
-	15750 3900 15850 3900
-Connection ~ 15850 3900
+	750  5550 850  5550
+Connection ~ 850  5550
 Wire Wire Line
-	15750 3700 15850 3700
-Connection ~ 15850 3700
+	750  5350 850  5350
+Connection ~ 850  5350
 Wire Wire Line
-	15750 3500 15850 3500
-Connection ~ 15850 3500
+	750  5150 850  5150
+Connection ~ 850  5150
 Wire Wire Line
-	15750 3300 15850 3300
-Connection ~ 15850 3300
+	750  4950 850  4950
+Connection ~ 850  4950
 Wire Wire Line
-	15750 3100 15850 3100
-Connection ~ 15850 3100
+	750  4750 850  4750
+Connection ~ 850  4750
 Wire Wire Line
-	15750 2900 15850 2900
-Connection ~ 15850 2900
+	750  4550 850  4550
+Connection ~ 850  4550
 Wire Wire Line
-	15750 2700 15850 2700
-Connection ~ 15850 2700
+	750  4350 850  4350
+Connection ~ 850  4350
 Wire Wire Line
-	15750 3800 15900 3800
+	750  5450 900  5450
 Wire Wire Line
-	15750 3600 15900 3600
+	750  5250 900  5250
 Wire Wire Line
-	15750 3200 15900 3200
+	750  4850 900  4850
 Wire Wire Line
-	15750 3400 15900 3400
+	750  5050 900  5050
 Wire Wire Line
-	15900 3000 15750 3000
+	900  4650 750  4650
 Wire Wire Line
-	15900 2800 15750 2800
+	900  4450 750  4450
 Wire Wire Line
-	15900 2600 15750 2600
+	900  4250 750  4250
 $Comp
 L VCC #PWR0112
@@
 L VCC #PWR0113
 U 1 1 5747F5DB
-P 16350 2400
-F 0 "#PWR0113" H 16350 2250 50  0001 C CNN
-F 1 "VCC" H 16350 2550 50  0000 C CNN
-F 2 "" H 16350 2400 50  0000 C CNN
-F 3 "" H 16350 2400 50  0000 C CNN
-	1    16350 2400
+P 1350 4050
+F 0 "#PWR0113" H 1350 3900 50  0001 C CNN
+F 1 "VCC" H 1350 4200 50  0000 C CNN
+F 2 "" H 1350 4050 50  0000 C CNN
+F 3 "" H 1350 4050 50  0000 C CNN
+	1    1350 4050
 	1    0    0    -1
 $EndComp
 Wire Wire Line
-	17200 650  17300 650
+	950  1250 1050 1250
 Wire Wire Line
-	17300 650  17300 1750
+	1050 1250 1050 2350
 $Comp
 L GND-RESCUE-FreeDSP_SMD #PWR0114
 U 1 1 57483422
-P 17300 1750
-F 0 "#PWR0114" H 17300 1750 30  0001 C CNN
-F 1 "GND" H 17300 1680 30  0001 C CNN
-F 2 "" H 17300 1750 60  0000 C CNN
-F 3 "" H 17300 1750 60  0000 C CNN
-	1    17300 1750
+P 1050 2350
+F 0 "#PWR0114" H 1050 2350 30  0001 C CNN
+F 1 "GND" H 1050 2280 30  0001 C CNN
+F 2 "" H 1050 2350 60  0000 C CNN
+F 3 "" H 1050 2350 60  0000 C CNN
+	1    1050 2350
 	1    0    0    -1
 $EndComp
 Wire Wire Line
-	17200 1650 17300 1650
-Connection ~ 17300 1650
+	950  2250 1050 2250
+Connection ~ 1050 2250
 Wire Wire Line
-	17200 1550 17350 1550
+	950  2150 1100 2150
 Wire Wire Line
-	17200 1150 17350 1150
+	950  1750 1100 1750
 Wire Wire Line
-	17200 1250 17350 1250
+	950  1850 1100 1850
 Wire Wire Line
-	17350 850  17200 850
+	1100 1450 950  1450
 Wire Wire Line
-	17350 750  17200 750
+	1100 1350 950  1350
 Wire Wire Line
-	17200 1450 17350 1450
+	950  2050 1100 2050
 Wire Wire Line
-	17200 1350 17350 1350
+	950  1950 1100 1950
 Wire Wire Line
-	17200 1050 17350 1050
+	950  1650 1100 1650
 Wire Wire Line
-	17200 950  17350 950
+	950  1550 1100 1550
 $Comp
 L +5V #PWR0115
 U 1 1 5743BA29
-P 17200 550
-F 0 "#PWR0115" H 17200 400 50  0001 C CNN
-F 1 "+5V" H 17200 690 50  0000 C CNN
-F 2 "" H 17200 550 50  0000 C CNN
-F 3 "" H 17200 550 50  0000 C CNN
-	1    17200 550
+P 950 1150
+F 0 "#PWR0115" H 950 1000 50  0001 C CNN
+F 1 "+5V" H 950 1290 50  0000 C CNN
+F 2 "" H 950 1150 50  0000 C CNN
+F 3 "" H 950 1150 50  0000 C CNN
+	1    950  1150
 	1    0    0    -1
 $EndComp
@@
 L CONN_01X12 P12
 U 1 1 57441678
-P 17000 1100
-F 0 "P12" H 17000 1750 50  0000 C CNN
-F 1 "MM-12G" V 17100 1100 50  0000 C CNN
-F 2 "rklib:MM-12G" H 17000 1100 50  0001 C CNN
-F 3 "" H 17000 1100 50  0000 C CNN
-	1    17000 1100
+P 750 1700
+F 0 "P12" H 750 1050 50  0000 C CNN
+F 1 "MM-12G" V 850 1700 50  0000 C CNN
+F 2 "rklib:MM-12G" H 750 1700 50  0001 C CNN
+F 3 "" H 750 1700 50  0000 C CNN
+	1    750  1700
 	-1   0    0    -1
 $EndComp
 $Comp
-L GND-RESCUE-FreeDSP_SMD #PWR?
+L GND-RESCUE-FreeDSP_SMD #PWR0116
 U 1 1 5744CA0A
 P 2300 4150
-F 0 "#PWR?" H 2300 4150 30  0001 C CNN
+F 0 "#PWR0116" H 2300 4150 30  0001 C CNN
 F 1 "GND" H 2300 4080 30  0001 C CNN
 F 2 "" H 2300 4150 60  0000 C CNN
