File: SOURCES/FreeDSP_BAL.sch (KiCad schematic (older format))
At the start: 187 parts, among them IC1 AD8608ARZ, IC2 ADAU1701, IC3 24AA256, IC4 SN74LVC1G08DBVR, IC5 AD8608ARZ, IC6 AD8608ARZ, IC7 74HC4040D, P10 CONN_02X10, P11 MM-16G, P12 MM-12G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

Commit message: Updated Gerber and BOM
Other:
- moved on the sheet: C22, JP1, P11, P12
